File: kidslab-lamp/components-sheet.kicad_sch (KiCad schematic)
At the start: 25 parts, among them U2 LSM6DS3

Commit message: adding layout
Parts:
- BZ1: footprint (none) -> kidslab:Buzzer-FUET-4020
- C1, C3: now left out of the parts list
- D1, D2, D3, D4: footprint LED_SMD:LED_SK6812MINI_PLCC4_3.5x3.5mm_P1.75mm -> kidslab:WS2812B-Mini
Connections:
- net +3V3: now also C5.1, C5.1, C5.1, C5.1, D1.1 (VDD), D2.1 (VDD), D3.1 (VDD), D4.1 (VDD)
- net +5V: no longer C5.1, C5.1, C5.1, C5.1, D1.1 (VDD), D2.1 (VDD), D3.1 (VDD), D4.1 (VDD)

Commit message: fixing some silkscreen issues
Parts:
- C1, C3: now in the parts list
- renumbered C1 to J1
Changed lines of the file:
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@@
     )
   )
-  (symbol (lib_id "kidslab:pin_header_1x3") (at 127 105.41 270) (mirror x) (unit 1)
-    (in_bom no) (on_board yes) (dnp no)
-    (property "Reference" "C1" (at 128.2701 100.33 0)
-      (effects (font (size 1.27 1.27)) (justify left))
+  (symbol (lib_name "pin_header_1x3_1") (lib_id "kidslab:pin_header_1x3") (at 127 105.41 270) (mirror x) (unit 1)
+    (in_bom yes) (on_board yes) (dnp no)
+    (property "Reference" "C1" (at 127 100.33 90)
+      (effects (font (size 1.27 1.27)))
     )
     (property "Value" "pin_header_1x3" (at 121.92 111.76 0)
@@
         )
         (path "/3a714d6a-4fcb-43e8-9668-1af7c84d4f32/fe3cb29b-5b2e-4797-a46c-7df643663d6c"
-          (reference "C2") (unit 1)
+          (reference "J2") (unit 1)
         )
       )
@@
   )
   (symbol (lib_id "kidslab:pin_header_1x3") (at 163.83 105.41 270) (mirror x) (unit 1)
-    (in_bom no) (on_board yes) (dnp no)
-    (property "Reference" "C3" (at 165.1001 100.33 0)
-      (effects (font (size 1.27 1.27)) (justify left))
+    (in_bom yes) (on_board yes) (dnp no)
+    (property "Reference" "C3" (at 163.83 100.33 90)
+      (effects (font (size 1.27 1.27)))
     )
     (property "Value" "pin_header_1x3" (at 158.75 111.76 0)
@@
         )
         (path "/3a714d6a-4fcb-43e8-9668-1af7c84d4f32/fe3cb29b-5b2e-4797-a46c-7df643663d6c"
-          (reference "C3") (unit 1)
+          (reference "J3") (unit 1)
         )
       )
@@
   (symbol (lib_id "kidslab:HY-4A") (at 80.01 106.68 180) (unit 1)
     (in_bom yes) (on_board yes) (dnp no)
-    (property "Reference" "C1" (at 80.01 115.57 0)
-      (effects (font (size 1.27 1.27)))
-    )
-    (property "Value" "HY-4A" (at 80.01 113.03 0)
+    (property "Reference" "J1" (at 80.01 111.76 0)
+      (effects (font (size 1.27 1.27)))
+    )
+    (property "Value" "HY-4A" (at 77.47 105.41 90)
       (effects (font (size 1.27 1.27)))
     )
@@
       (project "kidslab-lamp"
         (path "/3a714d6a-4fcb-43e8-9668-1af7c84d4f32/fe3cb29b-5b2e-4797-a46c-7df643663d6c"
-          (reference "C1") (unit 1)
-        )
-      )
+          (reference "J1") (unit 1)
+        )
+      )

Commit message: fixing component attributes, moving v1 gerber files
Parts:
- C1, C3: now left out of the parts list
Changed lines of the file:
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@@
   )
   (symbol (lib_name "pin_header_1x3_1") (lib_id "kidslab:pin_header_1x3") (at 127 105.41 270) (mirror x) (unit 1)
-    (in_bom yes) (on_board yes) (dnp no)
+    (in_bom no) (on_board yes) (dnp no)
     (property "Reference" "C1" (at 127 100.33 90)
       (effects (font (size 1.27 1.27)))
@@
   )
   (symbol (lib_id "kidslab:pin_header_1x3") (at 163.83 105.41 270) (mirror x) (unit 1)
-    (in_bom yes) (on_board yes) (dnp no)
+    (in_bom no) (on_board yes) (dnp no)
     (property "Reference" "C3" (at 163.83 100.33 90)
       (effects (font (size 1.27 1.27)))
