File: kicad-nerdYcontroller/peripherals.kicad_sch (KiCad schematic)
At the start: 7 parts, among them J301 Conn_02x03_Odd_Even, J302 Conn_02x03_Odd_Even, U301 LSM6DS3TR-C

Commit message: Adding KiCad files for first controller production.
Parts:
- removed C301, C302: 100nF, Capacitor_SMD:C_0603_1608Metric, symbol kidslab:C-100nF-0603-50V
- added 3V3, GND301, VBUS301: kroko_doubleedge, kidslab:DoubleEdge, symbol kidslab:Double Kroko Edge Connector
- added A301, A302, A303, A304: arrow, kidslab:Kroko_Arrow, symbol kidslab:arrow
- added BZ301: Buzzer-FUET-5020, kidslab:FUET-5020, symbol kidslab:Buzzer-Fuet-5020
- added C301, C302: 100nF, Capacitor_SMD:C_0402_1005Metric, symbol kidslab:C-100nF-0402-25V
- added C303, C305: 1uF, Capacitor_SMD:C_0603_1608Metric, symbol kidslab:C-1uF-0603-25V_1
- added C304: 100nF, Capacitor_SMD:C_0603_1608Metric, symbol kidslab:C-100nF-0603-50V
- added D301: KT-0603R, LED_SMD:LED_0603_1608Metric, symbol kidslab:LED - RED - 0603
- added GP0, GP1, GP19, GP2, GP22, GP3: kroko_edge, kidslab:Edgeconnector, symbol kidslab:kroko_edge
- added J303: ZX-HY2.0-4PLT, kidslab:ZX-HY2.0-4PLT, symbol kidslab:ZX-HY2.0-4PLT Grove connector
- added J304: HLE-115-02-F-DV, kidslab:SAMTEC_HLE-115-02-F-DV, symbol kidslab:HLE-115-02-F-DV
- added Q301: DDTC113ZCA, Package_TO_SOT_SMD:SOT-23, symbol kidslab:DDTC113ZCA
- added R303, R304, R305, R306: 1M, Resistor_SMD:R_0603_1608Metric, symbol kidslab:R-1M-0603
- added R307: 1k, Resistor_SMD:R_0603_1608Metric, symbol kidslab:R-1k-0603
- added R308: 33k, Resistor_SMD:R_0603_1608Metric, symbol kidslab:R-33k-0603
- added R309: 330R, Resistor_SMD:R_0603_1608Metric, symbol kidslab:R-330R-0603
- added U302: LMA3722T421-OA5, kidslab:LMA3722T421-OA5, symbol kidslab:LMA3722T421-OA5
- J301, J302: footprint Connector_PinHeader_2.54mm:PinHeader_2x03_P2.54mm_Vertical_SMD -> kidslab:PinHeader_2x03_P2.54mm_Vertical_SMD
- U301: footprint Package_LGA:LGA-14_3x2.5mm_P0.5mm_LayoutBorder3x4y -> kidslab:LGA-14_3x2.5mm_P0.5mm_LayoutBorder3x4y
Connections:
- net +3V3_in: now also 3V3.1, BZ301.1 (+), C301.2, C302.2, C304.1, C305.1, J303.3 (Pin_3), J304.02, J304.08, J304.14, J304.20, R308.1, U302.2 (VDD)
- net GND: now also C301.1, C302.1, C304.2, C305.2, D301.1 (K), GND301.1, J303.4 (Pin_4), J304.01, J304.07, J304.13, J304.19, J304.27, Q301.2 (E), R303.2, R304.2, R305.2, R306.2, R307.2, U302.3 (GND), U302.4 (GND)
- net +5V renamed VBUS
- net VBUS: now also J304.28, VBUS301.1
- net GP2/SERVO_2 renamed GP4/SERVO_2
- net GP3/SERVO_3 renamed GP5/SERVO_3
- net GP5/INTR renamed GP13/INTR
- net GP6/SDA1 renamed GP6/IMU_SDA
- net GP7/SCL1 renamed GP7/IMU_SCL
- new net: C303.1, U302.1 (out)
- new net: D301.2 (A), R309.2
- new net: BZ301.2 (-), Q301.3 (C)
- new net GP0: GP0.1, J304.04
- new net GP1: GP1.1, J304.03
- new net GP14/ArrowLeft: A301.1, J304.23, R303.1
- new net GP15/ArrowUp: A302.1, J304.24, R304.1
- new net GP16/ArrowRight: A303.1, J304.26, R305.1
- new net GP17/ArrowDown: A304.1, J304.25, R306.1
- new net GP18: J304.12
- new net GP19: GP19.1, J304.09
- new net GP2: GP2.1, J304.06
- new net GP20/Buzzer: Q301.1 (B)
- new net GP21: J304.11
- new net GP22: GP22.1, J304.10
- new net GP23: J304.15
- new net GP24: J304.16
- new net GP25/LED: J304.17, R309.1
- new net GP26: J304.21
- new net GP27: J304.18
- new net GP28: J304.22
- new net GP29/MIC_OUT: C303.2, R307.1, R308.2
- new net GP3: GP3.1, J304.05
- new net GP8/Grove_D1: J303.2 (Pin_2)
- new net GP9/Grove_D0: J303.1 (Pin_1)
- new net SWCLK: J304.29
- new net SWD: J304.30
- no-connect marks 1 -> 3
Other:
- note added: "Buzzer"
- note added: "Grove Connector"
- note added: "LED Matrix"
- note added: "Microphone"
- note added: "Pin Header"
- note added: "Status LED"
- note added: "Touch Pads"
- moved on the sheet: J301, J302, R302
